Commit message: Imported upstream version '1.1.0' of 'upstream'

File: urdf/common.xacro (robot description, xacro)
@@ -8,4 +8,5 @@
   <!-- All units in m-kg-s-radians unit system -->
   <xacro:property name="M_PI" value="3.1415926535897932" />
+  <xacro:property name="WHEEL_VELOCITY_LIMIT" value="90" />
   <!-- Inertial macros. Units are kg*m^2 -->
   <xacro:macro name="box_inertia" params="m x y z">

File: urdf/raspimouse.urdf.xacro (robot description, xacro)
@@ -11,6 +11,9 @@
   <xacro:arg name="jointstate" default="true" />
   <xacro:arg name="robot_namespace" default="/" />
-  <xacro:arg name="diffdrive_namespace" default="/" />
   <xacro:arg name="sensor_namespace" default="raspimouse_on_gazebo" />
+  <xacro:arg name="use_gazebo" default="false" />
+  <xacro:arg name="use_rgb_camera" default="false" />
+  <xacro:arg name="gz_control_config_package" default="" />
+  <xacro:arg name="gz_control_config_file_path" default="" />
   <material name="black">
     <color rgba="0.2 0.2 0.2 1.0"/>
@@ -21,6 +24,8 @@
   <xacro:include filename="$(find raspimouse_description)/urdf/wheel/wheel.urdf.xacro" />
   <xacro:include filename="$(find raspimouse_description)/urdf/wheel/diffdrive.gazebo.xacro" />
+  <xacro:include filename="$(find raspimouse_description)/urdf/wheel/diffdrive.gazebo_ros2_control.xacro" />
   <xacro:include filename="$(find raspimouse_description)/urdf/sensors/lightsens.urdf.xacro" />
   <xacro:include filename="$(find raspimouse_description)/urdf/sensors/lidar.urdf.xacro" />
+  <xacro:include filename="$(find raspimouse_description)/urdf/sensors/rgb_camera.xacro" />
   <!-- =============== Link & Joint =============== -->
   <!-- Base -->
@@ -81,4 +86,17 @@
   </xacro:if>
   <!-- =============== Gazebo =============== -->
+  <xacro:rgb_camera_settings
+    use_gazebo="$(arg use_gazebo)"
+    use_rgb_camera="$(arg use_rgb_camera)" />
+  <xacro:if value="$(arg use_gazebo)">
+    <xacro:gazebo_diffdrive_settings
+      use_gazebo="$(arg use_gazebo)"
+      config_file_package="$(arg gz_control_config_package)"
+      config_file_path="$(arg gz_control_config_file_path)" />
+    <xacro:diffdrive_gazebo_ros2_control_settings
+      name_hardware="GazeboSystem"
+      name_right_wheel_joint="right_wheel_joint"
+      name_left_wheel_joint="left_wheel_joint" />
+  </xacro:if>
   <xacro:if value="$(arg gazebo_plugin)">
     <gazebo>
@@ -113,7 +131,4 @@
       <xacro:lidar_gazebo sensor_link_name="$(arg lidar_frame)" base_rad="0" rad_range="6.28" min_range="0.15" max_range="12" />
     </xacro:if>
-    <!-- DiffDriveController -->
-    <xacro:diffdrive_gazebo publish_tf="$(arg tf)" publish_jointstate="$(arg jointstate)"
-      robot_namespace="$(arg diffdrive_namespace)" />
   </xacro:if>
   <raspimouse_on_gazebo/>

File: urdf/wheel/diffdrive.gazebo.xacro (robot description, xacro)
@@ -2,43 +2,19 @@
 <robot name="diffdrive_gazebo" xmlns:xacro="http://ros.org/wiki/xacro">
   <xacro:include filename="$(find raspimouse_description)/urdf/common.xacro" />
-  <xacro:macro name="diffdrive_gazebo" params="publish_tf publish_jointstate robot_namespace">
+  <xacro:macro name="gazebo_diffdrive_settings"
+    params="use_gazebo
+            config_file_package
+            config_file_path
+            ">
     <gazebo>
-      <plugin name="differential_drive_controller" filename="libgazebo_ros_diff_drive.so">
-        <!-- Name of robot namespace of DiffDriveController -->
-        <robotNamespace>${robot_namespace}</robotNamespace>
-        <alwaysOn>true</alwaysOn>
-        <updateRate>50</updateRate>
-        <!-- Set to true to swap right and left wheels, defaults to true -->
-        <legacyMode>false</legacyMode>
-        <rosDebugLevel>na</rosDebugLevel>
-        <!-- Name of left joint, defaults to `left_joint` -->
-        <leftJoint>left_wheel_joint</leftJoint>
-        <!-- Name of right joint, defaults to `right_joint` -->
-        <rightJoint>right_wheel_joint</rightJoint>
-        <robotBaseFrame>base_footprint</robotBaseFrame>
-        <!-- Topic to receive geometry_msgs/Twist message commands, defaults to `cmd_vel` -->
-        <commandTopic>cmd_vel</commandTopic>
-        <!-- Topic to publish nav_msgs/Odometry messages, defaults to `odom` -->
-        <odometryTopic>odom</odometryTopic>
-        <!-- Odometry frame, defaults to `odom` -->
-        <odometryFrame>odom</odometryFrame>
-        <!-- Odometry source, 0 for ENCODER, 1 for WORLD, defaults to WORLD -->
-        <odometrySource>world</odometrySource>
-        <!-- Phisical wheel params -->
-        <wheelSeparation>${wheel_separation}</wheelSeparation>
-        <wheelDiameter>${wheel_radius*2.0}</wheelDiameter>
-        <!-- Maximum torque which the wheels can produce, in Nm, defaults to 5 Nm -->
-        <wheelTorque>500</wheelTorque>
-        <!-- Wheel acceleration, in rad/s^2, defaults to 0.0 rad/s^2 -->
-        <wheelAcceleration>0</wheelAcceleration>
-        <!-- Set to true to publish /odom (nav_msgs::Odometry), defaults to true -->
-        <publishTf>${publish_tf}</publishTf>
-        <!-- Set to true to publish transforms for the wheel links, defaults to false -->
-        <publishWheelTF>${publish_tf}</publishWheelTF>
-        <!-- Set to true to publish transforms for the odometry, defaults to true -->
-        <publishOdomTF>${publish_tf}</publishOdomTF>
-        <!-- Set to true to publish sensor_msgs/JointState on /joint_states for the wheel joints, defaults to false -->
-        <publishWheelJointState>${publish_jointstate}</publishWheelJointState>
-      </plugin>
+      <xacro:if value="${use_gazebo}">
+        <plugin filename="libign_ros2_control-system.so" name="ign_ros2_control::IgnitionROS2ControlPlugin">
+          <ros>
+            <remapping>diff_drive_controller/cmd_vel_unstamped:=cmd_vel</remapping>
+            <remapping>diff_drive_controller/odom:=odom</remapping>
+          </ros>
+          <parameters>$(find ${config_file_package})/${config_file_path}</parameters>
+        </plugin>
+      </xacro:if>
     </gazebo>
   </xacro:macro>

File: urdf/wheel/wheel.urdf.xacro (robot description, xacro)
@@ -8,5 +8,5 @@
     <parent link="${parent}"/>
     <child link="${prefix}_wheel"/>
-    <limit effort="70" velocity="15"/>
+    <limit effort="70" velocity="${WHEEL_VELOCITY_LIMIT}"/>
     <safety_controller  k_velocity="10" />
     <dynamics damping="1.0" friction="1.0" />
