Commit message: Imported upstream version '2.0.0' of 'upstream'

File: urdf/sensors/lidar.gazebo.xacro (robot description, xacro)
@@ -5,5 +5,5 @@
       <sensor type="gpu_lidar" name="${sensor_link_name}_sensor">
         <pose relative_to='${sensor_link_name}'>0 0 0 0 0 0</pose>
-        <ignition_frame_id>${sensor_link_name}</ignition_frame_id>
+        <gz_frame_id>${sensor_link_name}</gz_frame_id>
         <frame_id>${sensor_link_name}</frame_id>
         <topic>scan</topic>

File: urdf/sensors/lightsens.urdf.xacro (robot description, xacro)
@@ -14,6 +14,6 @@
           <box size="0.01 0.005 0.007" />
         </geometry>
-        <material name="Gray">
-          <color rgba="0.2 0.2 0.2 1" />
+        <material name="Red">
+          <color rgba="1.0 0.0 0.0 1" />
         </material>
       </visual>

File: urdf/sensors/rgb_camera.xacro (robot description, xacro)
@@ -30,5 +30,5 @@
       <xacro:if value="${use_gazebo}">
         <gazebo>
-          <plugin filename="ignition-gazebo-sensors-system" name="ignition::gazebo::systems::Sensors">
+          <plugin filename="gz-sim-sensors-system" name="gz::sim::systems::Sensors">
             <render_engine>ogre2</render_engine>
           </plugin>
@@ -38,5 +38,5 @@
             <update_rate>30.0</update_rate>
             <always_on>true</always_on>
-            <ignition_frame_id>camera_link</ignition_frame_id>
+            <gz_frame_id>camera_link</gz_frame_id>
             <xacro:if value="${camera_downward}">
               <pose>0 0 0 0 ${DOWNWARD_CAMERA_ANGLE} 0</pose>

File: urdf/wheel/diffdrive.gazebo.xacro (robot description, xacro)
@@ -9,7 +9,7 @@
     <gazebo>
       <xacro:if value="${use_gazebo}">
-        <plugin filename="libign_ros2_control-system.so" name="ign_ros2_control::IgnitionROS2ControlPlugin">
+        <plugin filename="libgz_ros2_control-system.so" name="gz_ros2_control::GazeboSimROS2ControlPlugin">
           <ros>
-            <remapping>diff_drive_controller/cmd_vel_unstamped:=cmd_vel</remapping>
+            <remapping>diff_drive_controller/cmd_vel:=cmd_vel</remapping>
             <remapping>diff_drive_controller/odom:=odom</remapping>
           </ros>

File: urdf/wheel/diffdrive.gazebo_ros2_control.xacro (robot description, xacro)
@@ -8,5 +8,5 @@
     <ros2_control name="${name_hardware}" type="system">
       <hardware>
-        <plugin>ign_ros2_control/IgnitionSystem</plugin>
+        <plugin>gz_ros2_control/GazeboSimSystem</plugin>
       </hardware>
       <joint name="${name_right_wheel_joint}">
